File: HagiwoHatNoise.kicad_pcb (KiCad board)
At the start: 2 copper layers, 30 x 106 mm, 37 parts, among them J3 Eurorack_Power_10pin_Unshroud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, J6 TRIG, J7 DECAY CV, J8 TUNE CV, J9 OUT, Q1 2SC1815

Commit message: v1.1 ready for final check
Parts:
- C6: footprint Capacitor_THT:CP_Radial_D4.0mm_P1.50mm -> Capacitor_THT:CP_Radial_D4.0mm_P2.00mm
- J3: moved to B.Cu
- Q1: footprint Package_TO_SOT_THT:TO-92_Inline -> Package_TO_SOT_THT:TO-92L_Inline_Wide
- RV1, RV2, RV3: value 100k -> 100k B
- moved J3 10.2 mm to (61.0, 110.9)
- moved Q1 1.65 mm to (55.0, 104.3)
Routing:
- net Net-(J9-SIG): track 76.9 -> 59.2 mm, vias 2 -> 1
- net Net-(D1-A): track 111.8 -> 99.7 mm
- net Net-(R7-Pad1): track 37.2 -> 26.0 mm
- net Net-(Q1-C): track 58.8 -> 47.8 mm
- net D5: track 92.7 -> 103.0 mm, vias 0 -> 4
- net +12V: track 22.4 -> 32.0 mm
- net Net-(R1-Pad1): track 15.7 -> 22.7 mm
- net +5V: track 106.1 -> 112.4 mm
- net A5: track 78.1 -> 83.7 mm
- net D3: track 36.2 -> 40.8 mm
- net A0: track 8.74 -> 4.61 mm
- net Net-(R3-Pad1): track 16.7 -> 18.8 mm
- net A3: track 18.2 -> 17.1 mm
- net A1: track 11.6 -> 10.6 mm
- net A6: track 67.0 -> 66.2 mm, vias 0 -> 2
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Other:
- board text added: "V1.1"
- board text removed: "V1.0"
