File: HagiwoHatNoise.kicad_sch (KiCad schematic)
At the start: 37 parts, among them J1 Trig, J2 Decay CV, J3 Tune CV, J4 Eurorack_Power_16pin_Shrouded, J5 Out, Q1 2SC1815

Commit message: v1.0 ready for production
Parts:
- removed J1: Trig, Library:EighthInch_PJ398SM_T_TN_S, symbol Connector_Audio:AudioJack2_SwitchT
- removed J2: Decay CV, Library:EighthInch_PJ398SM_T_TN_S, symbol Connector_Audio:AudioJack2_SwitchT
- removed J3: Tune CV, Library:EighthInch_PJ398SM_T_TN_S, symbol Connector_Audio:AudioJack2_SwitchT
- removed J4: Eurorack_Power_16pin_Shrouded, Library:Pins_2x08_2.54mm_TH_EuroPower_Shrouded_Minimal, symbol PCM_4ms_Connector:Eurorack_Power_16pin_Shrouded
- removed J5: Out, Library:EighthInch_PJ398SM_T_TN_S, symbol Connector_Audio:AudioJack2_SwitchT
- added J3: Eurorack_Power_10pin_Unshrouded, Library:IDC-Header_2x05_P2.54mm_Vertical_Euro_Power_Striped_ThickerText, symbol PCM_4ms_Connector:Eurorack_Power_10pin_Unshrouded
- added J6: TRIG, Library:EighthInch_PJ398SM_3mmNPTH, symbol PCM_4ms_Jack:3.5mm_Mono_Switched_sm
- added J7: DECAY CV, Library:EighthInch_PJ398SM_3mmNPTH, symbol PCM_4ms_Jack:3.5mm_Mono_Switched_sm
- added J8: TUNE CV, Library:EighthInch_PJ398SM_3mmNPTH, symbol PCM_4ms_Jack:3.5mm_Mono_Switched_sm
- added J9: OUT, Library:EighthInch_PJ398SM_3mmNPTH, symbol PCM_4ms_Jack:3.5mm_Mono_Switched_sm
- C1: renamed from C5; value 2.2uF (225) -> 2.2uF; Silkscreen Value (none) -> 225▼
- C2: renamed from C3; value 22nF (223) -> 22nF; Silkscreen Value (none) -> 223▼
- C3: renamed from C4; value 3.3nF (332) -> 3.3nF; Silkscreen Value (none) -> 332▼
- C4: renamed from C1; value 100pF (101) -> 100pF; Silkscreen Value (none) -> 101▲
- C5: renamed from C6; value 100nF (104) -> 100nF; Silkscreen Value (none) -> 104▲
- C6: renamed from C7; footprint Capacitor_THT:CP_Radial_D6.3mm_P2.50mm -> Capacitor_THT:CP_Radial_D4.0mm_P1.50mm; Silkscreen Value (none) -> 10uF▶
- C7: renamed from C2; value 100pF (101) -> 100pF; Silkscreen Value (none) -> 101▲
- D1: renamed from D7; value LED_Filled -> LED
- D2: renamed from D1; footprint Diode_THT:D_DO-35_SOD27_P7.62mm_Horizontal -> Library:D_DO-35_SOD27_P7.62mm_Horizontal_Widened_No_K; Silkscreen Value (none) -> B43
- D3: renamed from D2; footprint Diode_THT:D_DO-35_SOD27_P7.62mm_Horizontal -> Library:D_DO-35_SOD27_P7.62mm_Horizontal_Widened_No_K; Silkscreen Value (none) -> B43
- D4: renamed from D3; footprint Diode_THT:D_DO-35_SOD27_P7.62mm_Horizontal -> Library:D_DO-35_SOD27_P7.62mm_Horizontal_Widened_No_K; Silkscreen Value (none) -> B43
- D5: renamed from D4; footprint Diode_THT:D_DO-35_SOD27_P7.62mm_Horizontal -> Library:D_DO-35_SOD27_P7.62mm_Horizontal_Widened_No_K; Silkscreen Value (none) -> B43
- D6: renamed from D5; footprint Diode_THT:D_DO-35_SOD27_P7.62mm_Horizontal -> Library:D_DO-35_SOD27_P7.62mm_Horizontal_Widened_No_K; Silkscreen Value (none) -> B43
- D7: renamed from D6; footprint Diode_THT:D_DO-35_SOD27_P7.62mm_Horizontal -> Library:D_DO-35_SOD27_P7.62mm_Horizontal_Widened_No_K; Silkscreen Value (none) -> B43
- Q1: Silkscreen Value (none) -> 2SC1815▲
- R1: value 1K -> 1k
- R10: renamed from R5; value 1K -> 1k
- R11: renamed from R8; value 100K -> 100k
- R12: renamed from R6; value 1K -> 1k
- R13: renamed from R9; value 100K -> 100k
- R3: renamed from R2; value 1K -> 1k
- R4: renamed from R12; value 2.7K -> 2.7k
- R5: renamed from R13; value 100K -> 100k
- R6: renamed from R10; value 33K -> 33k
- R7: renamed from R3; value 1K -> 1k
- R8: renamed from R4; value 1K -> 1k
- R9: renamed from R7; value 100K -> 100k
- RV1: renamed from Tune1; value 100K -> 100k
- RV2: renamed from Tone1; value 100K -> 100k
- RV3: renamed from Decay1; value 100K -> 100k
- renumbered R11 to R2
Connections:
- net +12V: now also J3.1 (+12V), J3.2 (+12V)
- net GND: now also J3.3 (GND), J3.4 (GND), J3.5 (GND), J3.6 (GND), J3.7 (GND), J3.8 (GND), J6.3 (SW), J7.3 (SW), J8.3 (SW), J9.3 (SW)
- net at C1.2: now also J9.1 (SIG)
- net at R10.1: now also J7.1 (SIG)
- net at R12.1: now also J8.1 (SIG)
- net at R8.1: now also J6.1 (SIG)
- new net -12V: J3.10 (-12V), J3.9 (-12V)
Other:
- note removed: "5v from Arduino or directly from 5V rail? caps on 12V rail?"
- note removed: "Patch submodule uses 22uF ceramic here"
- moved on the sheet: C1, C5, C6

Commit message: latest updates
Changed lines of the file:
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@@
 	)
 	(junction
+		(at 118.11 106.68)
+		(diameter 0)
+		(color 0 0 0 0)
+	)
+	(junction
 		(at 81.28 90.17)
 		(diameter 0)
@@
 	(wire
 		(pts
+			(xy 111.76 106.68) (xy 118.11 106.68)
+		)
+		(stroke
+			(width 0)
+			(type default)
+		)
+	)
+	(wire
+		(pts
 			(xy 27.94 25.4) (xy 34.29 25.4)
 		)
@@
 	)
 	(symbol
+		(lib_id "PCM_4ms_Power-symbol:PWR_FLAG")
+		(at 111.76 106.68 0)
+		(mirror y)
+		(unit 1)
+		(exclude_from_sim no)
+		(in_bom yes)
+		(on_board yes)
+		(dnp no)
+		(property "Reference" "#FLG03"
+			(at 111.76 104.775 0)
+			(effects
+				(font
+					(size 1.27 1.27)
+				)
+				(hide yes)
+			)
+		)
+		(property "Value" "PWR_FLAG"
+			(at 111.76 100.33 0)
+			(effects
+				(font
+					(size 1.27 1.27)
+				)
+			)
+		)
+		(property "Footprint" ""
+			(at 111.76 106.68 0)
+			(effects
+				(font
+					(size 1.27 1.27)
+				)
+				(hide yes)
+			)
+		)
+		(property "Datasheet" ""
+			(at 111.76 106.68 0)
+			(effects
+				(font
+					(size 1.27 1.27)
+				)
+				(hide yes)
+			)
+		)
+		(property "Description" ""
+			(at 111.76 106.68 0)
+			(effects
+				(font
+					(size 1.27 1.27)
+				)
+				(hide yes)
+			)
+		)
+		(pin "1"
+		)
+		(instances
+			(project "HagiwoHatNoise"
+				(path "/599a98da-a4a2-4635-97eb-f901b14811e2"
+					(reference "#FLG03")
+					(unit 1)
+				)
+			)
+		)
+	)
+	(symbol
 		(lib_id "power:+12V")
 		(at 120.65 19.05 0)
@@
 		(on_board yes)
 		(dnp no)
-		(fields_autoplaced yes)
 		(property "Reference" "#FLG01"
 			(at 111.76 98.425 0)
@@
 		)
 		(property "Value" "PWR_FLAG"
-			(at 111.76 101.6 0)
+			(at 111.76 102.87 0)
 			(effects
 				(font

Commit message: v1.1 ready for final check
Parts:
- C3: Silkscreen Value 332▼ -> 332▶
- C5: Silkscreen Value 104▲ -> ◀104
- C6: footprint Capacitor_THT:CP_Radial_D4.0mm_P1.50mm -> Capacitor_THT:CP_Radial_D4.0mm_P2.00mm
- Q1: footprint Package_TO_SOT_THT:TO-92_Inline -> Package_TO_SOT_THT:TO-92L_Inline_Wide; Silkscreen Value 2SC1815▲ -> 2SC1815▶
- RV1, RV2, RV3: value 100k -> 100k B
Changed lines of the file:
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@@
 			)
 		)
-		(property "Footprint" "Capacitor_THT:CP_Radial_D4.0mm_P1.50mm"
+		(property "Footprint" "Capacitor_THT:CP_Radial_D4.0mm_P2.00mm"
 			(at 164.7952 104.14 0)
 			(effects
@@
 			)
 		)
-		(property "Silkscreen Value" "104▲"
+		(property "Silkscreen Value" "◀104"
 			(at 143.51 100.33 0)
 			(effects
@@
 			)
 		)
-		(property "Value" "100k"
+		(property "Value" "100k B"
 			(at 21.59 62.2299 0)
 			(effects
@@
 			)
 		)
-		(property "Value" "100k"
+		(property "Value" "100k B"
 			(at 21.59 26.6699 0)
 			(effects
@@
 			)
 		)
-		(property "Value" "100k"
+		(property "Value" "100k B"
 			(at 21.59 44.4499 0)
 			(effects
@@
 			)
 		)
-		(property "Silkscreen Value" "332▼"
+		(property "Silkscreen Value" "332▶"
 			(at 181.61 54.61 0)
 			(effects
@@
 			)
 		)
-		(property "Footprint" "Package_TO_SOT_THT:TO-92_Inline"
+		(property "Footprint" "Package_TO_SOT_THT:TO-92L_Inline_Wide"
 			(at 202.565 22.86 0)
 			(effects
@@
 			)
 		)
-		(property "Silkscreen Value" "2SC1815▲"
+		(property "Silkscreen Value" "2SC1815▶"
 			(at 200.66 27.94 90)
 			(effects
