File: HagiwoHatNoise_Panel.kicad_pcb (KiCad board)
At the start: 2 copper layers, 30 x 128.5 mm, 9 parts

Commit message: v1.1 ready for final check
Parts:
- added REF**: Faceplate_Hole_LED_3mm, PCM_4ms_Faceplate:Faceplate_Hole_LED_3mm, F.Cu at (73.4, 147.6)
